File: PCB/Pi_zero_header.kicad_sch (KiCad schematic)
At the start: 93 parts, among them J1 Raspberry_Pi_2_3, J2 USB_C_Receptacle_USB2.0, J3 Screw_Terminal_01x02, J4 Screw_Terminal_01x02, J5 Conn_02x04_Top_Bottom, J6 Conn_01x07, J7 Conn_01x02, J8 Conn_02x03_Top_Bottom, J9 Conn_01x02, SW1 SW_Push, SW2 SW_Push, U1 RP2040, U2 W25Q128JVS, U3 TB6612FNG, U4 TPS630701RNMR, U5 TPS630701RNMR, U6 PQ25792RQMR, Y2 12M

Commit message: Another changes
Parts:
- C51: footprint Capacitor_SMD:C_0805_2012Metric -> Capacitor_SMD:C_0603_1608Metric
Other:
- moved on the sheet: C22, C24, C26, C27, C35, C36
Changed lines of the file:
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@@
   (junction (at 384.81 193.04) (diameter 0) (color 0 0 0 0)
   )
-  (junction (at 148.59 63.5) (diameter 0) (color 0 0 0 0)
-  )
   (junction (at 309.88 26.67) (diameter 0) (color 0 0 0 0)
   )
@@
   (junction (at 99.06 265.43) (diameter 0) (color 0 0 0 0)
   )
+  (junction (at 148.59 63.5) (diameter 0) (color 0 0 0 0)
+  )
   (junction (at 218.44 119.38) (diameter 0) (color 0 0 0 0)
   )
   (junction (at 130.81 161.29) (diameter 0) (color 0 0 0 0)
   )
+  (junction (at 137.16 63.5) (diameter 0) (color 0 0 0 0)
+  )
   (junction (at 140.97 173.99) (diameter 0) (color 0 0 0 0)
   )
@@
   (junction (at 287.02 26.67) (diameter 0) (color 0 0 0 0)
   )
+  (junction (at 137.16 71.12) (diameter 0) (color 0 0 0 0)
+  )
   (junction (at 360.68 182.88) (diameter 0) (color 0 0 0 0)
   )
@@
   (junction (at 195.58 77.47) (diameter 0) (color 0 0 0 0)
   )
-  (junction (at 137.16 71.12) (diameter 0) (color 0 0 0 0)
-  )
   (junction (at 309.88 46.99) (diameter 0) (color 0 0 0 0)
   )
@@
   (junction (at 27.94 234.95) (diameter 0) (color 0 0 0 0)
   )
-  (junction (at 137.16 63.5) (diameter 0) (color 0 0 0 0)
-  )
   (junction (at 294.64 46.99) (diameter 0) (color 0 0 0 0)
   )
@@
     (stroke (width 0) (type default))
   )
+  (wire (pts (xy 148.59 63.5) (xy 160.02 63.5))
+    (stroke (width 0) (type default))
+  )
   (wire (pts (xy 384.81 73.66) (xy 369.57 73.66))
     (stroke (width 0) (type default))
@@
     (stroke (width 0) (type default))
   )
-  (wire (pts (xy 148.59 63.5) (xy 160.02 63.5))
+  (wire (pts (xy 137.16 63.5) (xy 148.59 63.5))
     (stroke (width 0) (type default))
   )
@@
     (stroke (width 0) (type default))
   )
-  (wire (pts (xy 137.16 63.5) (xy 148.59 63.5))
-    (stroke (width 0) (type default))
-  )
   (wire (pts (xy 294.64 46.99) (xy 294.64 60.96))
     (stroke (width 0) (type default))
@@
     )
   )
-  (symbol (lib_id "Device:C") (at 40.64 39.37 0) (unit 1)
+  (symbol (lib_id "Device:C") (at 53.34 39.37 0) (unit 1)
     (in_bom yes) (on_board yes) (dnp no) (fields_autoplaced)
-    (property "Reference" "C22" (at 44.45 38.1 0)
+    (property "Reference" "C22" (at 57.15 38.1 0)
       (effects (font (size 1.27 1.27)) (justify left))
     )
-    (property "Value" "100n" (at 44.45 40.64 0)
+    (property "Value" "100n" (at 57.15 40.64 0)
       (effects (font (size 1.27 1.27)) (justify left))
     )
-    (property "Footprint" "Capacitor_SMD:C_0402_1005Metric" (at 41.6052 43.18 0)
+    (property "Footprint" "Capacitor_SMD:C_0402_1005Metric" (at 54.3052 43.18 0)
       (effects (font (size 1.27 1.27)) hide)
     )
-    (property "Datasheet" "~" (at 40.64 39.37 0)
+    (property "Datasheet" "~" (at 53.34 39.37 0)
       (effects (font (size 1.27 1.27)) hide)
     )
@@
     )
   )
-  (symbol (lib_id "Device:C") (at 148.59 67.31 0) (unit 1)
+  (symbol (lib_id "Device:C") (at 137.16 67.31 0) (unit 1)
     (in_bom yes) (on_board yes) (dnp no)
-    (property "Reference" "C35" (at 152.4 66.04 0)
+    (property "Reference" "C35" (at 140.97 66.04 0)
       (effects (font (size 1.27 1.27)) (justify left))
     )
-    (property "Value" "100n" (at 152.4 68.58 0)
+    (property "Value" "100n" (at 140.97 68.58 0)
       (effects (font (size 1.27 1.27)) (justify left))
     )
-    (property "Footprint" "Capacitor_SMD:C_0402_1005Metric" (at 149.5552 71.12 0)
+    (property "Footprint" "Capacitor_SMD:C_0402_1005Metric" (at 138.1252 71.12 0)
       (effects (font (size 1.27 1.27)) hide)
     )
-    (property "Datasheet" "~" (at 148.59 67.31 0)
+    (property "Datasheet" "~" (at 137.16 67.31 0)
       (effects (font (size 1.27 1.27)) hide)
     )
@@
     )
   )
-  (symbol (lib_id "Device:C") (at 29.21 69.85 0) (unit 1)
+  (symbol (lib_id "Device:C") (at 40.64 69.85 0) (unit 1)
     (in_bom yes) (on_board yes) (dnp no) (fields_autoplaced)
-    (property "Reference" "C26" (at 33.02 68.58 0)
+    (property "Reference" "C26" (at 44.45 68.58 0)
       (effects (font (size 1.27 1.27)) (justify left))
     )
-    (property "Value" "100n" (at 33.02 71.12 0)
+    (property "Value" "100n" (at 44.45 71.12 0)
       (effects (font (size 1.27 1.27)) (justify left))
     )
-    (property "Footprint" "Capacitor_SMD:C_0402_1005Metric" (at 30.1752 73.66 0)
+    (property "Footprint" "Capacitor_SMD:C_0402_1005Metric" (at 41.6052 73.66 0)
       (effects (font (size 1.27 1.27)) hide)
     )
-    (property "Datasheet" "~" (at 29.21 69.85 0)
+    (property "Datasheet" "~" (at 40.64 69.85 0)
       (effects (font (size 1.27 1.27)) hide)
     )
@@
     )
   )
-  (symbol (lib_id "Device:C") (at 137.16 67.31 0) (mirror y) (unit 1)
+  (symbol (lib_id "Device:C") (at 148.59 67.31 0) (mirror y) (unit 1)
     (in_bom yes) (on_board yes) (dnp no) (fields_autoplaced)
-    (property "Reference" "C36" (at 140.97 66.04 0)
+    (property "Reference" "C36" (at 152.4 66.04 0)
       (effects (font (size 1.27 1.27)) (justify right))
     )
-    (property "Value" "47u" (at 140.97 68.58 0)
+    (property "Value" "47u" (at 152.4 68.58 0)
       (effects (font (size 1.27 1.27)) (justify right))
     )
-    (property "Footprint" "Capacitor_SMD:C_1206_3216Metric" (at 136.1948 71.12 0)
+    (property "Footprint" "Capacitor_SMD:C_1206_3216Metric" (at 147.6248 71.12 0)
       (effects (font (size 1.27 1.27)) hide)
     )
-    (property "Datasheet" "~" (at 137.16 67.31 0)
+    (property "Datasheet" "~" (at 148.59 67.31 0)
       (effects (font (size 1.27 1.27)) hide)
     )
@@
       (effects (font (size 1.27 1.27)) (justify left))
     )
-    (property "Footprint" "Capacitor_SMD:C_0805_2012Metric" (at 103.8352 242.57 0)
+    (property "Footprint" "Capacitor_SMD:C_0603_1608Metric" (at 103.8352 242.57 0)
       (effects (font (size 1.27 1.27)) hide)
     )
@@
     )
   )
-  (symbol (lib_id "Device:C") (at 40.64 69.85 0) (unit 1)
+  (symbol (lib_id "Device:C") (at 29.21 69.85 0) (unit 1)
     (in_bom yes) (on_board yes) (dnp no) (fields_autoplaced)
-    (property "Reference" "C27" (at 44.45 68.58 0)
+    (property "Reference" "C27" (at 33.02 68.58 0)
       (effects (font (size 1.27 1.27)) (justify left))
     )
-    (property "Value" "22u" (at 44.45 71.12 0)
+    (property "Value" "22u" (at 33.02 71.12 0)
       (effects (font (size 1.27 1.27)) (justify left))
     )
-    (property "Footprint" "Capacitor_SMD:C_0805_2012Metric" (at 41.6052 73.66 0)
+    (property "Footprint" "Capacitor_SMD:C_0805_2012Metric" (at 30.1752 73.66 0)
       (effects (font (size 1.27 1.27)) hide)
     )
-    (property "Datasheet" "~" (at 40.64 69.85 0)
+    (property "Datasheet" "~" (at 29.21 69.85 0)
       (effects (font (size 1.27 1.27)) hide)
     )
@@
     )
   )
-  (symbol (lib_id "Device:C") (at 53.34 39.37 0) (unit 1)
+  (symbol (lib_id "Device:C") (at 40.64 39.37 0) (unit 1)
     (in_bom yes) (on_board yes) (dnp no) (fields_autoplaced)
-    (property "Reference" "C24" (at 57.15 38.1 0)
+    (property "Reference" "C24" (at 44.45 38.1 0)
       (effects (font (size 1.27 1.27)) (justify left))
     )
-    (property "Value" "22u" (at 57.15 40.64 0)
+    (property "Value" "22u" (at 44.45 40.64 0)
       (effects (font (size 1.27 1.27)) (justify left))
     )
-    (property "Footprint" "Capacitor_SMD:C_0805_2012Metric" (at 54.3052 43.18 0)
+    (property "Footprint" "Capacitor_SMD:C_0805_2012Metric" (at 41.6052 43.18 0)
       (effects (font (size 1.27 1.27)) hide)
     )
-    (property "Datasheet" "~" (at 53.34 39.37 0)
+    (property "Datasheet" "~" (at 40.64 39.37 0)
       (effects (font (size 1.27 1.27)) hide)
     )

Commit message: Another changes...
Parts:
- added R23, R9: 10k, Resistor_SMD:R_0402_1005Metric, symbol Device:R
Connections:
- net +3V3: now also R23.1, R9.1
- net CE_N_RPI: now also U1.9 (GPIO7); no longer U1.8 (GPIO6)
- net MISO_RPi: now also U1.11 (GPIO8); no longer U1.9 (GPIO7)
- net MOSI_RPi: now also U1.12 (GPIO9); no longer U1.11 (GPIO8)
- net SCLK_RPi: now also J6.3 (Pin_3), U1.13 (GPIO10); no longer U1.12 (GPIO9)
- net SCL_PWR: now also R9.2
- net SDA_PWR: now also R23.2
- new net INT_N_PWR: U1.8 (GPIO6)
Other:
- moved on the sheet: J8

Commit message: Bruuuhhhh...
Parts:
- H1, H2, H3, H4: footprint MountingHole:MountingHole_2.7mm_M2.5 -> MountingHole:MountingHole_2.7mm
- R11: value 6k04 -> 3k
Connections:
- net AIN1: now also U1.30 (GPIO19); no longer U1.32 (GPIO21)
- net AIN2: now also U1.31 (GPIO20); no longer U1.34 (GPIO22)
- net BIN1: now also U1.32 (GPIO21); no longer U1.35 (GPIO23)
- net BIN2: now also U1.34 (GPIO22); no longer U1.36 (GPIO24)
- net PWMA: now also U1.28 (GPIO17); no longer U1.30 (GPIO19)
- net PWMB: now also U1.29 (GPIO18); no longer U1.31 (GPIO20)
- net STBY_N: now also U1.35 (GPIO23); no longer U1.37 (GPIO25)
- net VBUS: now also U6.8 (VAC2), U6.9 (VAC1)
- net XIN: now also Y2.1; no longer Y2.3
- net at C3.1, R5.1: now also Y2.3; no longer Y2.1
- net at U1.18 (GPIO15): now also J8.4 (Pin_4); no longer D2.1 (K)
- net at U1.27 (GPIO16): now also J8.1 (Pin_1)
- new net: D2.1 (K), U1.37 (GPIO25)
Other:
- moved on the sheet: D2, R22, Y2
