File: PCB/Pi_zero_header.kicad_pcb (KiCad board)
At the start: 2 copper layers, 30 x 65 mm, 95 parts, among them J1 Raspberry_Pi_2_3, J2 USB_C_Receptacle_USB2.0, J3 Screw_Terminal_01x02, J4 Screw_Terminal_01x02, J5 Conn_02x04_Top_Bottom, J6 Conn_01x07, J7 Conn_01x02, J8 Conn_02x03_Top_Bottom, J9 Conn_01x02, SW1 SW_Push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

Commit message: Finally picked inductors
Parts:
- added JP1: SolderJumper_2_Open, Jumper:SolderJumper-2_P1.3mm_Open_RoundedPad1.0x1.5mm, F.Cu at (74.0, 100.8)
- added JP2: SolderJumper_2_Open, Jumper:SolderJumper-2_P1.3mm_Open_RoundedPad1.0x1.5mm, F.Cu at (74.9, 101.8)
- added JP3: SolderJumper_2_Open, Jumper:SolderJumper-2_P1.3mm_Open_RoundedPad1.0x1.5mm, F.Cu at (74.0, 102.7)
- added R24: 6k04, Resistor_SMD:R_0402_1005Metric, F.Cu at (77.5, 101.8)
- added R25: 10k5, Resistor_SMD:R_0402_1005Metric, F.Cu at (77.5, 102.8)
- added R26: 5k1, Resistor_SMD:R_0402_1005Metric, F.Cu at (62.0, 111.3)
- added R27: 5k1, Resistor_SMD:R_0402_1005Metric, F.Cu at (62.0, 113.2)
- L1: footprint Inductor_SMD:L_1008_2520Metric -> Inductor_SMD:L_Vishay_IFSC-1515AH_4x4x1.8mm
- L2, L3: value 1.5u -> 1u; footprint Inductor_SMD:L_1008_2520Metric -> Inductor_SMD:L_Vishay_IFSC-1515AH_4x4x1.8mm
- moved R11 13.7 mm to (77.5, 100.8), turned to 0 degrees
- moved C29 3.03 mm to (67.2, 91.7)
- moved C30 3.03 mm to (67.2, 89.7)
- moved C26 3.03 mm to (63.9, 99.2)
- moved C27 3.03 mm to (62.7, 102.0)
- moved C31 3.03 mm to (65.0, 94.8)
- moved C32 3.03 mm to (62.5, 99.8)
- moved C33 3.03 mm to (62.5, 96.7)
- moved C35 3.03 mm to (63.9, 97.3)
- moved C36 3.03 mm to (61.5, 94.5)
- moved D1 3.03 mm to (63.8, 105.5)
- moved J7 3.03 mm to (59.8, 91.0)
- moved J9 3.03 mm to (63.5, 91.0)
- moved L1 3.03 mm to (60.2, 98.2)
- moved R7 3.03 mm to (64.8, 105.5)
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Connections:
- J2 pad A5: unconnected-(J2-CC1-PadA5) -> Net-(J2-CC1)
- J2 pad B5: unconnected-(J2-CC2-PadB5) -> Net-(J2-CC2)
- J6 pad 3: /SCLK_RPi -> Net-(J6-Pin_3)
- R11 pad 1: Net-(U6-PROG) -> Net-(JP1-A)
- U1 pad 11: /MISO_RPi -> /SCLK_RPi
- U1 pad 12: /MOSI_RPi -> unconnected-(U1-GPIO9-Pad12)
- U1 pad 13: /SCLK_RPi -> Net-(J6-Pin_3)
- U1 pad 6: /CE_N_PWR -> /INT_N_PWR
- U1 pad 7: /QON_N_PWR -> /CE_N_RPI
- U1 pad 8: /INT_N_PWR -> /MISO_RPi
- U1 pad 9: /CE_N_RPI -> /MOSI_RPi
- U6 pad 12: /QON_N_PWR -> unconnected-(U6-QON_N-Pad12)
- U6 pad 13: /CE_N_PWR -> GND
- U6 pad 20: Net-(U6-PROG) -> Net-(JP1-B)
- U6 pad 21: /INT_N -> /INT_N_PWR

Commit message: Another changes to PCB
Parts:
- J1: moved to B.Cu
- moved C47 49.7 mm to (45.2, 141.5)
- moved C48 49.7 mm to (45.2, 139.5)
- moved C49 49.7 mm to (51.0, 134.8)
- moved C50 49.7 mm to (46.2, 137.0)
- moved C51 49.7 mm to (46.2, 134.0)
- moved C52 49.7 mm to (46.0, 131.5)
- moved C53 49.7 mm to (46.0, 129.5)
- moved L3 49.7 mm to (43.8, 135.5)
- moved R18 49.7 mm to (48.8, 138.0)
- moved R19 49.7 mm to (49.0, 133.0)
- moved R20 49.7 mm to (51.0, 133.0)
- moved R21 49.7 mm to (49.0, 132.0)
- moved U5 49.7 mm to (48.8, 135.5)
- moved J1 48.2 mm to (44.8, 106.6)
- moved C4 29.5 mm to (73.3, 72.8)
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Connections:
- JP2 pad 1: Net-(JP2-A) -> Net-(JP1-A)
- JP2 pad 2: Net-(JP1-B) -> Net-(JP2-B)
- JP3 pad 1: Net-(JP3-A) -> Net-(JP1-A)
- JP3 pad 2: Net-(JP1-B) -> Net-(JP3-B)
- R11 pad 1: Net-(JP1-A) -> Net-(JP1-B)
- R24 pad 1: Net-(JP2-A) -> Net-(JP2-B)
- R25 pad 1: Net-(JP3-A) -> Net-(JP3-B)
- U6 pad 20: Net-(JP1-B) -> Net-(JP1-A)

Commit message: Bruuuuh, me mad...
Parts:
- added JP4: SolderJumper_2_Open, Jumper:SolderJumper-2_P1.3mm_Open_RoundedPad1.0x1.5mm, F.Cu at (42.8, 87.7)
- moved H1 64.7 mm to (66.5, 114.0), turned to 180 degrees
- moved H2 64.7 mm to (43.5, 114.0), turned to 180 degrees
- moved C47 61.3 mm to (53.0, 80.8), turned to 90 degrees
- moved H3 60.1 mm to (66.5, 56.0), turned to 180 degrees
- moved H4 60.1 mm to (43.5, 56.0), turned to 180 degrees
- moved C48 59.1 mm to (51.0, 80.8), turned to 90 degrees
- moved R18 57.0 mm to (49.5, 81.0), turned to 90 degrees
- moved C49 56.2 mm to (46.2, 78.8), turned to 180 degrees
- moved R26 55.9 mm to (48.8, 56.5), turned to 180 degrees
- moved J2 55.0 mm to (55.0, 56.2), turned to 180 degrees
- moved U5 54.5 mm to (47.0, 81.0), turned to -90 degrees
- moved R20 54.4 mm to (44.5, 79.0), turned to 90 degrees
- moved R27 54.0 mm to (48.8, 57.5), turned to 180 degrees
- moved C50 53.5 mm to (48.5, 83.5), turned to 180 degrees
- moved R19 52.2 mm to (44.5, 81.0), turned to 90 degrees
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Connections:
- C51 pad 1: +3V3 -> Net-(JP4-A)
- C52 pad 1: +3V3 -> Net-(JP4-A)
- C53 pad 1: +3V3 -> Net-(JP4-A)
- R19 pad 1: +3V3 -> Net-(JP4-A)
- R21 pad 1: +3V3 -> Net-(JP4-A)
- U5 pad 7: +3V3 -> Net-(JP4-A)
- U5 pad 8: +3V3 -> Net-(JP4-A)

Commit message: Getting somewhere...
Parts:
- moved C17 42.1 mm to (45.2, 90.0), turned to 180 degrees
- moved C20 41.3 mm to (45.8, 88.2), turned to 180 degrees
- moved U3 38.4 mm to (47.0, 83.0)
- moved C18 27.8 mm to (52.2, 79.5), turned to 90 degrees
- moved C19 24.8 mm to (54.0, 79.0), turned to 90 degrees
- moved C53 21.8 mm to (58.0, 98.0), turned to -90 degrees
- moved JP4 20.4 mm to (60.6, 97.5), turned to 0 degrees
- moved R21 18.9 mm to (54.0, 96.8), turned to 180 degrees
- moved C52 18.9 mm to (56.0, 98.0), turned to -90 degrees
- moved R20 18.4 mm to (52.0, 95.8), turned to 180 degrees
- moved R19 17.5 mm to (54.0, 95.8), turned to 180 degrees
- moved C49 16.2 mm to (51.8, 94.0), turned to -90 degrees
- moved C51 15.7 mm to (56.5, 94.8), turned to 90 degrees
- moved L3 14.5 mm to (60.2, 93.2), turned to -90 degrees
- moved U5 14.1 mm to (54.0, 93.2), turned to 0 degrees
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
Commit message: Another commit :)
Parts:
- removed C4, C48: 10u, Capacitor_SMD:C_0805_2012Metric
- removed C44, C52: 22u, Capacitor_SMD:C_0805_2012Metric
- C41, C47: value 10u -> 22u
- moved JP4 3.67 mm to (57.0, 97.9), turned to -90 degrees
- moved C47 2.76 mm to (52.0, 90.5)
- moved C53 2.24 mm to (60.0, 97.0), turned to 0 degrees
- moved C45 1.58 mm to (60.0, 88.2), turned to 0 degrees
- moved C41 1.12 mm to (60.5, 80.8), turned to 0 degrees
- moved C49 0.75 mm to (52.5, 94.0)
- moved C50 0.75 mm to (57.2, 91.8)
- moved C51 0.75 mm to (57.2, 94.8)
- moved L2 0.75 mm to (61.0, 84.5)
- moved L3 0.75 mm to (61.0, 93.2)
- moved R18 0.75 mm to (54.8, 90.8)
- moved R19 0.75 mm to (54.8, 95.8)
- moved R20 0.75 mm to (52.8, 95.8)
- moved R21 0.75 mm to (54.8, 96.8)
- moved U5 0.75 mm to (54.8, 93.2)

Commit message: Bruh, I forgor...
Parts:
- J2: footprint Connector_USB:USB_C_Receptacle_GCT_USB4105-xx-A_16P_TopMnt_Horizontal -> Connector_USB:USB_C_Receptacle_GCT_USB4110
- J3, J4: value Screw_Terminal_01x02 -> Conn_01x02; footprint TerminalBlock_TE-Connectivity:TerminalBlock_TE_282834-2_1x02_P2.54mm_Horizontal -> Connector_PinHeader_2.54mm:PinHeader_1x02_P2.54mm_Vertical
- moved J6 161.8 mm to (29.8, 69.4)
- moved J5 136.9 mm to (21.5, 94.0)
- moved J8 136.9 mm to (28.4, 99.7)
- moved C10 21.5 mm to (87.5, 92.2)
- moved C11 21.5 mm to (88.7, 95.2)
- moved C12 21.5 mm to (88.7, 99.0)
- moved C13 21.5 mm to (84.0, 103.5)
- moved C14 21.5 mm to (78.2, 99.0)
- moved C15 21.5 mm to (78.2, 95.2)
- moved C16 21.5 mm to (90.0, 102.2)
- moved C2 21.5 mm to (79.7, 107.5)
- moved C3 21.5 mm to (85.2, 107.5)
- moved C5 21.5 mm to (75.2, 88.2)
- moved C6 21.5 mm to (85.0, 103.5)
- moved C7 21.5 mm to (82.7, 92.2)
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
Commit message: Still working on PCB...
Parts:
- moved SW1 20.2 mm to (76.2, 86.2), turned to 180 degrees
- moved C5 19.5 mm to (94.5, 85.5), turned to 0 degrees
- moved C2 18.0 mm to (75.2, 90.0), turned to 0 degrees
- moved R2 17.9 mm to (92.5, 85.5), turned to 180 degrees
- moved R1 16.7 mm to (90.5, 85.5), turned to 0 degrees
- moved Y2 16.4 mm to (75.2, 92.8), turned to -90 degrees
- moved C3 15.6 mm to (75.2, 95.5), turned to 180 degrees
- moved U2 15.3 mm to (94.0, 89.0), turned to 0 degrees
- moved SW2 14.6 mm to (76.2, 99.2), turned to 180 degrees
- moved J8 13.4 mm to (17.0, 106.8)
- moved R5 12.8 mm to (77.5, 94.0), turned to 90 degrees
- moved J6 12.1 mm to (29.2, 81.5)
- moved C14 11.8 mm to (83.8, 88.5), turned to 90 degrees
- moved C15 11.5 mm to (87.5, 88.5), turned to 90 degrees
- moved R23 11.4 mm to (85.5, 88.5), turned to -90 degrees
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Routing:
- net Net-(U6-SW2): track 0.00 -> 14.0 mm, vias 0 -> 2
- net Net-(U6-SW1): track 0.00 -> 14.0 mm, vias 0 -> 2
- net Net-(U6-BTST2): track 0.00 -> 6.65 mm, vias 0 -> 2
- net Net-(U6-BTST1): track 0.00 -> 5.59 mm, vias 0 -> 2

Commit message: Finally gonna rout'em
Parts:
- J5: value Conn_02x04_Top_Bottom -> Conn_02x04_Odd_Even
- moved R1 49.4 mm to (48.0, 110.8), turned to 180 degrees
- moved R2 48.8 mm to (45.0, 96.8), turned to -90 degrees
- moved U2 44.8 mm to (50.2, 98.5)
- moved C5 40.7 mm to (55.5, 97.0), turned to -90 degrees
- moved C15 39.5 mm to (50.8, 103.0), turned to 180 degrees
- moved SW1 39.2 mm to (48.8, 114.2), turned to -90 degrees
- moved R9 39.0 mm to (50.8, 104.0), turned to 0 degrees
- moved R23 38.5 mm to (50.8, 105.0), turned to 0 degrees
- moved C14 37.7 mm to (50.8, 106.8), turned to 180 degrees
- moved C7 35.2 mm to (56.0, 99.8), turned to 90 degrees
- moved R3 34.8 mm to (58.2, 99.0), turned to -90 degrees
- moved C2 34.2 mm to (52.2, 115.2), turned to 90 degrees
- moved C9 34.0 mm to (57.0, 99.8), turned to 90 degrees
- moved R4 33.7 mm to (59.2, 99.0), turned to -90 degrees
- moved C8 31.6 mm to (59.2, 101.0)
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Connections:
- J5 pad 2: GND -> +3V3
- J5 pad 3: Net-(J5-Pin_3) -> GND
- J5 pad 4: Net-(J5-Pin_4) -> GND
- J5 pad 5: +3V3 -> Net-(J5-Pin_5)
- J5 pad 6: GND -> Net-(J5-Pin_5)
- J5 pad 7: Net-(J5-Pin_3) -> Net-(J5-Pin_7)
- J5 pad 8: Net-(J5-Pin_4) -> Net-(J5-Pin_7)
- J8 pad 2: +5V -> Net-(J8-Pin_2)
- J8 pad 3: GND -> +5V
- J8 pad 4: Net-(J8-Pin_4) -> +5V
- J8 pad 5: +5V -> GND
- U1 pad 18: Net-(J8-Pin_4) -> Net-(J8-Pin_2)
- U1 pad 2: Net-(J5-Pin_3) -> Net-(J5-Pin_5)
- U1 pad 3: Net-(J5-Pin_4) -> Net-(J5-Pin_7)
Routing:
- net Net-(U6-SW2): track 14.0 -> 13.5 mm
- net Net-(U6-SW1): track 14.0 -> 13.5 mm
